File: test/test.kicad_pcb (KiCad board)
At the start: 2 copper layers, 60 x 60 mm, 24 parts, among them J1 Conn_Coaxial, J2 Conn_Coaxial, J3 Conn_01x02, J4 Conn_01x02, J5 Screw_Terminal_01x01, J6 Screw_Terminal_01x01, J7 Screw_Terminal_01x01, J8 Screw_Terminal_01x01, U1 OPA188xxD, U2 OPA188xxD

Commit message: PCB tracing done
Parts:
- C1, C2, R3: moved to B.Cu
- moved J2 229.0 mm to (13.1, 17.6), turned to 90 degrees
- moved J4 222.5 mm to (32.4, 23.0)
- moved J3 210.2 mm to (39.0, 29.9), turned to 180 degrees
- moved J1 207.7 mm to (13.2, 41.4), turned to 90 degrees
- moved R3 106.1 mm to (28.9, 35.5)
- moved C5 103.1 mm to (23.8, 37.9), turned to 90 degrees
- moved R2 102.2 mm to (28.6, 41.9)
- moved C2 102.2 mm to (24.2, 36.3), turned to 90 degrees
- moved C1 97.9 mm to (28.4, 37.2), turned to 180 degrees
- moved C6 97.2 mm to (33.5, 35.0), turned to 90 degrees
- moved R1 95.1 mm to (26.7, 40.4)
- moved U1 87.7 mm to (28.6, 36.5)
Routing:
- net +5V: track 2.27 -> 37.1 mm
- net -5V: track 2.77 -> 35.0 mm
- net Net-(J2-In): track 7.31 -> 38.7 mm
- net Net-(C1-Pad1): track 0.00 -> 26.2 mm, vias 0 -> 2
- net Net-(J1-In): track 0.00 -> 13.0 mm
- net Net-(C1-Pad2): track 0.00 -> 8.12 mm, vias 0 -> 1
- net Net-(U1--): track 0.00 -> 5.15 mm, vias 0 -> 1
- net GND: track 0.00 -> 4.92 mm, vias 0 -> 2
Other:
- board text added: "+5V"
- board text added: "-5V"
- board text added: "IN"
- board text added: "Made by BMSTU SAPR"
- board text added: "OUT"
