File: kek/kek.kicad_sch (KiCad schematic)
At the start: 26 parts, among them X1 B3P-VH

Commit message: new files
Connections:
- net OUT3: now also DA3.2 (IN+), R12.2, R13.2
Other:
- moved on the sheet: DA3, X1
